Commit message: updated code with error fixed

File: my_rb1_description/urdf/my_rb1_robot.urdf (robot description, URDF)
Before this commit: robot robot, 7 links, 6 joints
Links:
- link back_caster: mass None -> 0.5
- link base_link: mass 25 -> 20.5
- link front_caster: mass None -> 0.5
- link left_wheel: mass 0.5 -> 1.5
- link right_wheel: mass 0.5 -> 1.5
Joints:
- joint front_caster_wheel_joint: origin xyz=-0.1 0.0 -0.15 rpy=0 0 0 -> xyz=0.1 0.0 -0.15 rpy=0 0 0
- joint rear_caster_wheel_joint: origin xyz=0.1 0.0 -0.15 rpy=0 0 0 -> xyz=-0.1 0.0 -0.15 rpy=0 0 0
